File: hardware/dsi_bridge.kicad_sch (KiCad schematic)
At the start: 17 parts, among them J11 Conn_01x20_MountingPin, J12 Conn_01x20_MountingPin, U15 AP3032

Commit message: Removed old readme, added files.
Parts:
- C44: MPN CL05B104KB54PNC -> CL05B105KQ5NQNC
Changed lines of the file:
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@@
 			)
 		)
-		(property "MPN" "CL05B104KB54PNC"
+		(property "MPN" "CL05B105KQ5NQNC"
 			(at 87.63 68.58 0)
 			(effects
