File: hardware/usb.kicad_sch (KiCad schematic)
At the start: 43 parts, among them J10 Conn_01x01_Pin, J4 USB_A, J5 USB_A, J6 Conn_01x01_Pin, J7 Conn_01x01_Pin, J9 Conn_01x01_Pin, U3 USB2514B_Bi, U4 MIC2026-1xM, U5 USBLC6-2SC6, U6 USBLC6-2SC6, U8 USBLC6-2SC6, Y1 24Mhz

Commit message: Removed old readme, added files.
Parts:
- C12: MPN CL10A475MQ8NNNC -> CC0402MRX5R5BB475
- C30: MPN CL05B104KB54PNC -> CL05B105KQ5NQNC
Changed lines of the file:
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@@
 			)
 		)
-		(property "MPN" "CL05B104KB54PNC"
+		(property "MPN" "CL05B105KQ5NQNC"
 			(at 69.85 85.09 0)
 			(effects
@@
 			)
 		)
-		(property "MPN" "CL10A475MQ8NNNC"
+		(property "MPN" "CC0402MRX5R5BB475"
 			(at 55.88 60.96 0)
 			(effects
